Commit message: 修正步兵的模型坐标系

File: assets/drago_infantry/infantry.urdf (robot description, URDF)
Before this commit: robot infantry, 7 links, 6 joints
Links:
- link base_link: mass 4.01063271963356 -> 4.01063271963357
- link left_wheel: mass 0.576889812400611 -> 0.576889812400606
- link right_small_leg: mass 0.371276470595446 -> 0.371276470595448
- link right_wheel: mass 0.576889812400578 -> 0.576889812400577
Joints:
- joint left_leg: axis 0 0 1 -> 0 -1 0; origin xyz=-0.1774 0 0.082513 rpy=1.5708 0 1.5708 -> xyz=0.0774339304506741 0.166046528452957 0.112513103962355 rpy=0 0 0
- joint left_small_leg: axis 0 0 -1 -> 0 1 0; origin xyz=-0.205577835151384 -0.0954826905438838 -0.0526438005535146 rpy=0 0 0 -> xyz=-0.205577835151374 0.0095000000000004 -0.0629504066267599 rpy=0 0 0
- joint left_wheel: axis 0 0 -1 -> 0 1 0; origin xyz=0.240043707112295 -0.0830362491674771 -0.0310500000000015 rpy=0 0 0 -> xyz=0.240043707112258 0.0310500000000015 -0.083036249167477 rpy=0 0 0
- joint right_leg: axis 0 0 -1 -> 0 1 0; origin xyz=0.175 0 0.0825131039623545 rpy=1.5707963267949 0 1.5707963267949 -> xyz=0.0774339304506787 -0.186353471547043 0.112513103962355 rpy=0 0 0
- joint right_small_leg: axis 0 0 1 -> 0 -1 0; origin xyz=-0.205577835151344 -0.0629504066268236 0.0109999999999999 rpy=0 0 0 -> xyz=-0.20557783515135 -0.0109999999999999 -0.0629504066268527 rpy=0 0 0
- joint right_wheel: axis 0 0 1 -> 0 -1 0; origin xyz=0.240043707112294 -0.0830362491673799 0.0435500000000003 rpy=0 0 0 -> xyz=0.24004370711208 -0.0435500000000003 -0.0830362491679966 rpy=0 0 0
